File: snap_board.kicad_pcb (KiCad board)
At the start: 6 copper layers, 121 parts, among them U1 STM32MP157CAC3, U2 AS4C256M16D3LC-12BCN, U3 S40FC004C1B2C00000, U4 STPMIC1BPQR, U5 DF40C-70DP-0.4V(51), U6 DF40C-70DP-0.4V(51), U7 DF40C-70DP-0.4V(51), X1 32.768kHz, X2 24MHz

Commit message: ram complete
Parts:
- C30, C31, C32, C33: moved to F.Cu
- moved C30 81.6 mm to (101.7, 135.3), turned to 270 degrees
- moved C22 44.2 mm to (143.1, 127.8), turned to 180 degrees
- moved C32 41.6 mm to (139.5, 148.3), turned to 90 degrees
- moved C15 40.5 mm to (143.1, 126.7), turned to 180 degrees
- moved C33 30.1 mm to (160.8, 148.9), turned to 90 degrees
- moved C9 29.0 mm to (160.5, 126.2)
- moved C21 26.9 mm to (160.5, 127.4)
- moved C31 16.0 mm to (162.1, 128.9), turned to 90 degrees
Routing:
- net GND: track 130.5 -> 135.5 mm, vias 95 -> 97
- net PMIC_VOUT2_VDD_DDR: track 45.6 -> 46.3 mm, vias 22 -> 23

Commit message: modified sch and layout
Parts:
- removed Re: 56E, Resistor_SMD:R_0402_1005Metric
- added C63: 1uF, Capacitor_SMD:C_0402_1005Metric, F.Cu at (188.0, 72.5)
- added C64: 1uF, Capacitor_SMD:C_0402_1005Metric, F.Cu at (188.0, 74.5)
- added C65: 1uF, Capacitor_SMD:C_0402_1005Metric, F.Cu at (190.9, 72.5)
- added C66: 1uF, Capacitor_SMD:C_0402_1005Metric, F.Cu at (188.0, 76.4)
- added C67: 1uF, Capacitor_SMD:C_0402_1005Metric, F.Cu at (190.9, 74.5)
- added C68: 1uF, Capacitor_SMD:C_0402_1005Metric, F.Cu at (193.7, 72.5)
- added C69: 1uF, Capacitor_SMD:C_0402_1005Metric, F.Cu at (190.9, 76.4)
- added C70: 1uF, Capacitor_SMD:C_0402_1005Metric, F.Cu at (193.7, 74.5)
- added C71: 1uF, Capacitor_SMD:C_0402_1005Metric, F.Cu at (196.6, 72.5)
- added C72: 1uF, Capacitor_SMD:C_0402_1005Metric, F.Cu at (193.7, 76.4)
- added C73: 1uF, Capacitor_SMD:C_0402_1005Metric, F.Cu at (196.6, 74.5)
- added C74: 1uF, Capacitor_SMD:C_0402_1005Metric, F.Cu at (196.6, 76.4)
- added FID1: Fiducial, Fiducial:Fiducial_0.5mm_Mask1.5mm, F.Cu at (123.0, 68.0)
- added FID2: Fiducial, Fiducial:Fiducial_0.5mm_Mask1.5mm, F.Cu at (157.0, 68.5)
- added FID3: Fiducial, Fiducial:Fiducial_0.5mm_Mask1.5mm, F.Cu at (157.5, 115.0)
- added FID4: Fiducial, Fiducial:Fiducial_0.5mm_Mask1.5mm, B.Cu at (123.0, 68.0)
- added FID5: Fiducial, Fiducial:Fiducial_0.5mm_Mask1.5mm, B.Cu at (157.0, 68.5)
- added FID6: Fiducial, Fiducial:Fiducial_0.5mm_Mask1.5mm, B.Cu at (157.5, 115.0)
- added H1: MountingHole_Pad, MountingHole:MountingHole_2.2mm_M2, F.Cu at (118.0, 69.5)
- added H2: MountingHole_Pad, MountingHole:MountingHole_2.2mm_M2, F.Cu at (162.0, 69.5)
- added H3: MountingHole_Pad, MountingHole:MountingHole_2.2mm_M2, F.Cu at (162.0, 113.5)
- added H4: MountingHole_Pad, MountingHole:MountingHole_2.2mm_M2, F.Cu at (118.0, 113.5)
- added R16: 56E, Resistor_SMD:R_0402_1005Metric, B.Cu at (155.4, 88.0)
- U5, U6, U7: moved to B.Cu
- moved R44 146.7 mm to (126.7, 95.8), turned to 270 degrees
- moved R41 139.2 mm to (131.4, 95.9), turned to 270 degrees
- moved R45 138.9 mm to (127.8, 95.8), turned to 270 degrees
- moved R38 138.4 mm to (136.0, 102.5), turned to 180 degrees
- moved C42 137.2 mm to (132.4, 95.9), turned to 90 degrees
- moved R42 136.7 mm to (130.3, 95.9), turned to 270 degrees
- moved R43 135.8 mm to (136.0, 103.6), turned to 180 degrees
- moved R39 134.4 mm to (136.0, 98.2), turned to 180 degrees
- moved R37 133.0 mm to (136.0, 101.4), turned to 180 degrees
- moved R40 132.1 mm to (136.0, 99.2), turned to 180 degrees
- moved R36 131.2 mm to (136.0, 100.3), turned to 180 degrees
- moved U3 130.7 mm to (130.1, 102.5), turned to 270 degrees
- moved U5 88.6 mm to (120.5, 99.0), turned to 90 degrees
- moved U6 77.6 mm to (139.0, 112.5)
- moved C38 71.0 mm to (200.5, 80.2), turned to 180 degrees
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Routing:
- net SDMMC2_CMD: track 2.35 -> 29.7 mm, vias 0 -> 3
- net SDMMC2_D6: track 0.34 -> 27.1 mm, vias 1 -> 3
- net SDMMC2_CK: track 3.34 -> 28.5 mm, vias 0 -> 2
- net SDMMC2_D5: track 2.38 -> 22.7 mm, vias 0 -> 2
- net SDMMC2_D4: track 3.11 -> 22.6 mm, vias 0 -> 2
- net GND: track 135.5 -> 148.1 mm, vias 97 -> 104
- net SDMMC2_D3: track 2.76 -> 13.1 mm, vias 0 -> 2
- net SDMMC2_D2: track 2.38 -> 11.0 mm, vias 0 -> 2
- net SDMMC2_D0: track 3.26 -> 11.8 mm, vias 0 -> 2
- net SDMMC2_D7: track 2.94 -> 11.4 mm, vias 0 -> 2
- net SDMMC2_D1: track 2.61 -> 10.3 mm, vias 0 -> 2
- net PMIC_VOUT3_VDD: track 20.6 -> 28.2 mm, vias 12 -> 17
- net NRST: track 6.30 -> 10.7 mm
- net Net-(C42-Pad1): track 0.00 -> 3.44 mm
- net DSI_D0_N: track 3.16 -> 1.62 mm
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Other:
- board outline added: 50 x 50 mm
